File: rp6502.kicad_sch (KiCad schematic)
At the start: 51 parts, among them J1 AUDIO, J2 VGA, J3 REBOOT, J4 GPIO, J5 PIX, U1 W65C02S, U2 Pico RIA, U3 AS6C1008, U4 Pico VGA, U5 W65C22S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

Commit message: pcb complete
Parts:
- R18: value 8.06K -> 8.06k
- R21, R24: value 1.8K -> 1.8k
- SW1: renamed from J3; symbol Connector_Generic:Conn_02x01 -> Switch:SW_Push
- renumbered J4 to J1, J5 to J2, J2 to J3, J1 to J4
Connections:
- net A10: now also U8.2; no longer U8.3
- net A11: now also U8.3; no longer U8.4
- net A12: now also U8.4; no longer U8.5
- net A13: now also U8.5; no longer U8.6
- net A14: now also U8.6; no longer U8.11
- net A15: now also U8.11; no longer U8.12
- net A5: now also U6.12; no longer U6.9
- net A7: now also U6.9; no longer U6.12
- net A8: now also U8.12; no longer U8.1
- net A9: now also U8.1; no longer U8.2
- net IRQB: now also U7.13; no longer U7.10
- net RWB: now also U7.8; no longer U7.11
- net at U6.6: now also U7.11; no longer U7.8
- net at U6.2: now also U7.10; no longer U7.13
Other:
- moved on the sheet: J1, J2, J3, J4, JP1, JP2, R16, R17, U7C, U7D

Commit message: founders edition
Parts:
- U8: symbol 74xx:74LS30 -> RP6502:74HC30
Connections:
- net GND: now also U8.9 (NC)
Other:
- note added: "Power source is Pico USB"
- moved on the sheet: SW1
Changed lines of the file:
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@@
     (stroke (width 0) (type default))
   )
-  (wire (pts (xy 20.32 194.31) (xy 25.4 194.31))
+  (wire (pts (xy 20.32 176.53) (xy 25.4 176.53))
     (stroke (width 0) (type default))
   )
-  (wire (pts (xy 20.32 186.69) (xy 25.4 186.69))
+  (wire (pts (xy 20.32 189.23) (xy 25.4 189.23))
     (stroke (width 0) (type default))
   )
@@
     (stroke (width 0) (type default))
   )
-  (wire (pts (xy 20.32 189.23) (xy 25.4 189.23))
+  (wire (pts (xy 20.32 191.77) (xy 25.4 191.77))
     (stroke (width 0) (type default))
   )
@@
     (stroke (width 0) (type default))
   )
-  (wire (pts (xy 20.32 181.61) (xy 25.4 181.61))
+  (wire (pts (xy 20.32 184.15) (xy 25.4 184.15))
     (stroke (width 0) (type default))
   )
@@
     (stroke (width 0) (type default))
   )
-  (wire (pts (xy 99.06 106.68) (xy 92.71 106.68))
+  (wire (pts (xy 100.33 109.22) (xy 93.98 109.22))
     (stroke (width 0) (type default))
   )
@@
     (stroke (width 0) (type default))
   )
-  (wire (pts (xy 20.32 191.77) (xy 25.4 191.77))
+  (wire (pts (xy 20.32 194.31) (xy 25.4 194.31))
     (stroke (width 0) (type default))
   )
@@
     (stroke (width 0) (type default))
   )
-  (wire (pts (xy 20.32 179.07) (xy 25.4 179.07))
+  (wire (pts (xy 20.32 181.61) (xy 25.4 181.61))
     (stroke (width 0) (type default))
   )
@@
     (stroke (width 0) (type default))
   )
-  (wire (pts (xy 20.32 184.15) (xy 25.4 184.15))
+  (wire (pts (xy 20.32 186.69) (xy 25.4 186.69))
     (stroke (width 0) (type default))
   )
@@
     (stroke (width 0) (type default))
   )
-  (wire (pts (xy 20.32 176.53) (xy 25.4 176.53))
+  (wire (pts (xy 20.32 179.07) (xy 25.4 179.07))
+    (stroke (width 0) (type default))
+  )
+  (rectangle (start 290.83 182.88) (end 316.23 204.47)
     (stroke (width 0) (type default))
+    (fill (type none))
   )
   (text "Use 1% resistors for audio and video." (at 193.04 125.73 0)
     (effects (font (size 1.27 1.27)) (justify left bottom))
   )
+  (text "Power source\nis Pico USB" (at 297.18 187.96 0)
+    (effects (font (size 1.27 1.27)) (justify left bottom))
+  )
   (label "RED3" (at 163.83 57.15 0) (fields_autoplaced)
     (effects (font (size 1.27 1.27)) (justify left bottom))
@@
     (effects (font (size 1.27 1.27)) (justify right bottom))
   )
-  (label "A14" (at 20.32 189.23 0) (fields_autoplaced)
+  (label "A14" (at 20.32 191.77 0) (fields_autoplaced)
     (effects (font (size 1.27 1.27)) (justify left bottom))
   )
@@
     (effects (font (size 1.27 1.27)) (justify left bottom))
   )
-  (label "A12" (at 20.32 184.15 0) (fields_autoplaced)
+  (label "A12" (at 20.32 186.69 0) (fields_autoplaced)
     (effects (font (size 1.27 1.27)) (justify left bottom))
   )
@@
     (effects (font (size 1.27 1.27)) (justify left bottom))
   )
-  (label "A13" (at 20.32 186.69 0) (fields_autoplaced)
+  (label "A13" (at 20.32 189.23 0) (fields_autoplaced)
     (effects (font (size 1.27 1.27)) (justify left bottom))
   )
@@
     (effects (font (size 1.27 1.27)) (justify left bottom))
   )
-  (label "A15" (at 20.32 191.77 0) (fields_autoplaced)
+  (label "A15" (at 20.32 194.31 0) (fields_autoplaced)
     (effects (font (size 1.27 1.27)) (justify left bottom))
   )
@@
     (effects (font (size 1.27 1.27)) (justify left bottom))
   )
-  (label "A9" (at 20.32 176.53 0) (fields_autoplaced)
+  (label "A9" (at 20.32 179.07 0) (fields_autoplaced)
     (effects (font (size 1.27 1.27)) (justify left bottom))
   )
@@
     (effects (font (size 1.27 1.27)) (justify left bottom))
   )
-  (label "A11" (at 20.32 181.61 0) (fields_autoplaced)
+  (label "A11" (at 20.32 184.15 0) (fields_autoplaced)
     (effects (font (size 1.27 1.27)) (justify left bottom))
   )
@@
     (effects (font (size 1.27 1.27)) (justify right bottom))
   )
-  (label "A10" (at 20.32 179.07 0) (fields_autoplaced)
+  (label "A10" (at 20.32 181.61 0) (fields_autoplaced)
     (effects (font (size 1.27 1.27)) (justify left bottom))
   )
@@
     (effects (font (size 1.27 1.27)) (justify right bottom))
   )
-  (label "RUN" (at 99.06 106.68 180) (fields_autoplaced)
+  (label "RUN" (at 100.33 109.22 180) (fields_autoplaced)
     (effects (font (size 1.27 1.27)) (justify right bottom))
   )
@@
     (effects (font (size 1.27 1.27)) (justify right bottom))
   )
-  (label "A8" (at 20.32 194.31 0) (fields_autoplaced)
+  (label "A8" (at 20.32 176.53 0) (fields_autoplaced)
     (effects (font (size 1.27 1.27)) (justify left bottom))
   )
@@
     )
   )
-  (symbol (lib_id "power:PWR_FLAG") (at 289.56 57.15 0) (unit 1)
+  (symbol (lib_id "power:PWR_FLAG") (at 298.45 196.85 0) (unit 1)
     (in_bom yes) (on_board yes) (dnp no)
-    (property "Reference" "#FLG01" (at 289.56 55.245 0)
+    (property "Reference" "#FLG01" (at 298.45 194.945 0)
       (effects (font (size 1.27 1.27)) hide)
     )
-    (property "Value" "PWR_FLAG" (at 289.56 52.07 0)
+    (property "Value" "PWR_FLAG" (at 298.45 191.77 0)
       (effects (font (size 1.27 1.27)))
     )
-    (property "Footprint" "" (at 289.56 57.15 0)
+    (property "Footprint" "" (at 298.45 196.85 0)
       (effects (font (size 1.27 1.27)) hide)
     )
-    (property "Datasheet" "~" (at 289.56 57.15 0)
+    (property "Datasheet" "~" (at 298.45 196.85 0)
       (effects (font (size 1.27 1.27)) hide)
     )
@@
     )
   )
-  (symbol (lib_id "74xx:74LS30") (at 33.02 184.15 0) (unit 1)
+  (symbol (lib_id "RP6502:74HC30") (at 33.02 184.15 0) (unit 1)
     (in_bom yes) (on_board yes) (dnp no) (fields_autoplaced)
     (property "Reference" "U8" (at 33.02 171.45 0)
@@
     )
     (pin "1")
+    (pin "10")
     (pin "11")
     (pin "12")
+    (pin "13")
     (pin "2")
     (pin "3")
@@
     (pin "6")
     (pin "8")
+    (pin "9")
     (pin "14")
     (pin "7")
@@
     )
   )
-  (symbol (lib_id "power:PWR_FLAG") (at 299.72 57.15 180) (unit 1)
+  (symbol (lib_id "power:PWR_FLAG") (at 308.61 196.85 180) (unit 1)
     (in_bom yes) (on_board yes) (dnp no) (fields_autoplaced)
-    (property "Reference" "#FLG02" (at 299.72 59.055 0)
+    (property "Reference" "#FLG02" (at 308.61 198.755 0)
       (effects (font (size 1.27 1.27)) hide)
     )
-    (property "Value" "PWR_FLAG" (at 299.72 62.23 0)
+    (property "Value" "PWR_FLAG" (at 308.61 201.93 0)
       (effects (font (size 1.27 1.27)))
     )
-    (property "Footprint" "" (at 299.72 57.15 0)
+    (property "Footprint" "" (at 308.61 196.85 0)
       (effects (font (size 1.27 1.27)) hide)
     )
-    (property "Datasheet" "~" (at 299.72 57.15 0)
+    (property "Datasheet" "~" (at 308.61 196.85 0)
       (effects (font (size 1.27 1.27)) hide)
     )
@@
     )
   )
-  (symbol (lib_id "power:VBUS") (at 299.72 57.15 0) (unit 1)
+  (symbol (lib_id "power:VBUS") (at 308.61 196.85 0) (unit 1)
     (in_bom yes) (on_board yes) (dnp no) (fields_autoplaced)
-    (property "Reference" "#PWR05" (at 299.72 60.96 0)
+    (property "Reference" "#PWR05" (at 308.61 200.66 0)
       (effects (font (size 1.27 1.27)) hide)
     )
-    (property "Value" "VBUS" (at 299.72 52.07 0)
+    (property "Value" "VBUS" (at 308.61 191.77 0)
       (effects (font (size 1.27 1.27)))
     )
-    (property "Footprint" "" (at 299.72 57.15 0)
+    (property "Footprint" "" (at 308.61 196.85 0)
       (effects (font (size 1.27 1.27)) hide)
     )
-    (property "Datasheet" "" (at 299.72 57.15 0)
+    (property "Datasheet" "" (at 308.61 196.85 0)
       (effects (font (size 1.27 1.27)) hide)
     )
@@
     )
   )
-  (symbol (lib_id "power:GND") (at 289.56 57.15 0) (unit 1)
+  (symbol (lib_id "power:GND") (at 298.45 196.85 0) (unit 1)
     (in_bom yes) (on_board yes) (dnp no) (fields_autoplaced)
-    (property "Reference" "#PWR04" (at 289.56 63.5 0)
+    (property "Reference" "#PWR04" (at 298.45 203.2 0)
       (effects (font (size 1.27 1.27)) hide)
     )
-    (property "Value" "GND" (at 289.56 62.23 0)
+    (property "Value" "GND" (at 298.45 201.93 0)
       (effects (font (size 1.27 1.27)))
     )
-    (property "Footprint" "" (at 289.56 57.15 0)
+    (property "Footprint" "" (at 298.45 196.85 0)
       (effects (font (size 1.27 1.27)) hide)
     )
-    (property "Datasheet" "" (at 289.56 57.15 0)
+    (property "Datasheet" "" (at 298.45 196.85 0)
       (effects (font (size 1.27 1.27)) hide)
     )
@@
     )
   )
-  (symbol (lib_id "Switch:SW_Push") (at 87.63 106.68 0) (unit 1)
+  (symbol (lib_id "Switch:SW_Push") (at 88.9 109.22 0) (unit 1)
     (in_bom yes) (on_board yes) (dnp no)
-    (property "Reference" "SW1" (at 87.63 99.06 0)
+    (property "Reference" "SW1" (at 88.9 101.6 0)
       (effects (font (size 1.27 1.27)))
     )
-    (property "Value" "REBOOT" (at 87.63 101.6 0)
+    (property "Value" "REBOOT" (at 88.9 104.14 0)
       (effects (font (size 1.27 1.27)))
     )
-    (property "Footprint" "Button_Switch_THT:SW_Tactile_SKHH_Angled" (at 87.63 101.6 0)
+    (property "Footprint" "Button_Switch_THT:SW_Tactile_SKHH_Angled" (at 88.9 104.14 0)
       (effects (font (size 1.27 1.27)) hide)
     )
-    (property "Datasheet" "~" (at 87.63 101.6 0)
+    (property "Datasheet" "~" (at 88.9 104.14 0)
       (effects (font (size 1.27 1.27)) hide)
     )
@@
     )
   )
-  (symbol (lib_id "power:GND") (at 82.55 106.68 0) (unit 1)
+  (symbol (lib_id "power:GND") (at 83.82 109.22 0) (unit 1)
     (in_bom yes) (on_board yes) (dnp no) (fields_autoplaced)
-    (property "Reference" "#PWR0139" (at 82.55 113.03 0)
+    (property "Reference" "#PWR0139" (at 83.82 115.57 0)
       (effects (font (size 1.27 1.27)) hide)
     )
-    (property "Value" "GND" (at 82.55 111.76 0)
+    (property "Value" "GND" (at 83.82 114.3 0)
       (effects (font (size 1.27 1.27)) hide)
     )
-    (property "Footprint" "" (at 82.55 106.68 0)
+    (property "Footprint" "" (at 83.82 109.22 0)
       (effects (font (size 1.27 1.27)) hide)
     )
-    (property "Datasheet" "" (at 82.55 106.68 0)
+    (property "Datasheet" "" (at 83.82 109.22 0)
       (effects (font (size 1.27 1.27)) hide)
     )
