File: rp6502.kicad_sch (KiCad schematic)
At the start: 51 parts, among them J1 GPIO, J2 PIX, J3 VGA, J4 AUDIO, SW1 REBOOT, U1 W65C02S, U2 Pico RIA, U3 AS6C1008, U4 Pico VGA, U5 W65C22S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

Commit message: first assembly
Parts:
- J3: footprint Connector_Dsub:DSUB-15-HD_Female_Horizontal_P2.29x1.98mm_EdgePinOffset8.35mm_Housed_MountingHolesOffset10.89mm -> rp6502:DSUB-15-HD_Female_Horizontal_P2.29x2.54mm_EdgePinOffset8.35mm_Housed_MountingHolesOffset10.89mm
Changed lines of the file:
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@@
       (effects (font (size 1.27 1.27)))
     )
-    (property "Footprint" "Connector_Dsub:DSUB-15-HD_Female_Horizontal_P2.29x1.98mm_EdgePinOffset8.35mm_Housed_MountingHolesOffset10.89mm" (at 107.95 134.62 0)
+    (property "Footprint" "rp6502:DSUB-15-HD_Female_Horizontal_P2.29x2.54mm_EdgePinOffset8.35mm_Housed_MountingHolesOffset10.89mm" (at 107.95 134.62 0)
       (effects (font (size 1.27 1.27)) hide)
     )

Commit message: PTH slot increase for PCBWay
Parts:
- J4: footprint Connector_Audio:Jack_3.5mm_CUI_SJ1-3525N_Horizontal -> rp6502:Jack_3.5mm_CUI_SJ1-3525N_Horizontal
Changed lines of the file:
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@@
       (effects (font (size 1.27 1.27)))
     )
-    (property "Footprint" "Connector_Audio:Jack_3.5mm_CUI_SJ1-3525N_Horizontal" (at 130.81 193.04 0)
+    (property "Footprint" "rp6502:Jack_3.5mm_CUI_SJ1-3525N_Horizontal" (at 130.81 193.04 0)
       (effects (font (size 1.27 1.27)) hide)
     )

Commit message: revb
Parts:
- U2: value Pico RIA -> RP6502-RIA; footprint rp6502:DIP-40_W17.78mm_LongPads_PicoDebug -> rp6502:DIP-40_W17.78mm_LongPads
- U4: value Pico VGA -> RP6502-VGA
Connections:
- net GND: no longer U2.42 (GND)
- net SWCLK: no longer names the net of U2.41 (SWCLK)
- net SWCLK: no longer U4.29 (GP22)
- net SWDIO: no longer names the net of U2.43 (SWDIO)
- net SWDIO: no longer U4.34 (GP28)
- no-connect marks 21 -> 26
